File: DragonYUV.kicad_pcb (KiCad board)
At the start: 4 copper layers, 120 x 64.1 mm, 68 parts, among them IC1 74HCT273, IC10 74HCT32, IC12 CD4053, IC2 MC6847, IC3 74HCT00, IC4 74HCT20, IC5 74HCT86, IC6 74HCT393, IC7 74ALS74N, IC8 74HCT393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

Commit message: tidy up
Parts:
- U1: value AD624RJ -> AD724RJ
- moved R9 15.4 mm to (201.7, 83.3), turned to 90 degrees
- moved Q1 12.7 mm to (201.7, 81.0), turned to -90 degrees
- moved R7 11.2 mm to (202.7, 78.8), turned to 90 degrees
- moved R8 7.46 mm to (200.7, 77.0), turned to 90 degrees
- moved R10 2.95 mm to (184.2, 74.7)
- moved Q2 2.95 mm to (186.4, 75.5)
- moved R11 2.95 mm to (188.6, 75.6)
- moved TP2 2.74 mm to (166.7, 87.4)
- moved Q3 2.56 mm to (192.6, 72.6)
- moved R12 2.56 mm to (190.4, 71.7)
- moved R13 2.56 mm to (194.8, 72.7)
- moved FB1 2.03 mm to (207.4, 107.9), turned to -90 degrees
- moved TP3 1.59 mm to (167.4, 91.2)
- moved C10 0.38 mm to (196.6, 108.6)
Connections:
- net Net-(Q1-C) renamed /~{Y}
- RV1 pad 3: unconnected-(RV1-Pad3) -> GND
- RV2 pad 3: unconnected-(RV2-Pad3) -> GND
- RV3 pad 3: unconnected-(RV3-Pad3) -> GND
Routing:
- net ~{HS}: track 0.00 -> 81.8 mm, vias 0 -> 4
- net ~{NHS}: track 62.5 -> 139.5 mm, vias 0 -> 4
- net /~{VCLK}: track 0.00 -> 69.6 mm, vias 0 -> 4
- net Net-(IC3-Pad4): track 1.27 -> 61.7 mm, vias 0 -> 2
- net Net-(IC8A-MR): track 5.48 -> 62.6 mm, vias 0 -> 4
- net ~{FS}: track 146.2 -> 199.7 mm, vias 0 -> 2
- net VCLK: track 47.2 -> 93.4 mm, vias 1 -> 2
- net Net-(IC4-Pad1): track 1.27 -> 37.7 mm, vias 0 -> 4
- net Net-(IC7B-C): track 0.00 -> 34.9 mm, vias 0 -> 4
- net /FS': track 0.00 -> 31.6 mm, vias 0 -> 2
- net Net-(IC6B-Q0): track 0.00 -> 23.4 mm, vias 0 -> 2
- net Net-(IC7B-D): track 0.00 -> 23.3 mm, vias 0 -> 2
- net LUM CONTROL: track 33.1 -> 50.0 mm, vias 0 -> 2
- net Net-(IC9B-Q0): track 0.00 -> 15.3 mm, vias 0 -> 2
- net Net-(IC7B-Q): track 0.00 -> 14.0 mm, vias 0 -> 2
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