File: DragonYUV.kicad_sch (KiCad schematic)
At the start: 69 parts, among them IC1 74HCT273, IC10 74HCT32, IC12 CD4053, IC2 MC6847, IC3 74HCT00, IC4 74HCT20, IC5 74HCT86, IC6 74HCT393, IC7 74ALS74N, IC8 74HCT393, IC9 74HCT390, J1 Video Output, J2 Board Interconnect Male, Q1 MMBT4401, Q2 NPN, Q3 NPN, Q4 NPN, Q5 NPN, Q6 NPN, U1 AD624RJ, U2 74AHC1G04, Y1 4.433620MHz

Commit message: tidy up
Parts:
- U1: value AD624RJ -> AD724RJ
Connections:
- net GND: now also RV1.3, RV2.3, RV3.3
- net ~{Y}: now reaches Q1.1 (C), R14.2, R16.2, R20.2, R7.1
Changed lines of the file:
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@@
 		)
 	)
+	(label "~{Y}"
+		(at 274.32 35.56 0)
+		(fields_autoplaced yes)
+		(effects
+			(font
+				(size 1.27 1.27)
+			)
+			(justify left bottom)
+		)
+	)
 	(label "Y-B"
 		(at 273.05 85.09 0)
@@
 	)
 	(symbol
+		(lib_id "power:GND")
+		(at 312.42 49.53 0)
+		(unit 1)
+		(exclude_from_sim no)
+		(in_bom yes)
+		(on_board yes)
+		(dnp no)
+		(fields_autoplaced yes)
+		(property "Reference" "#PWR03"
+			(at 312.42 55.88 0)
+			(effects
+				(font
+					(size 1.27 1.27)
+				)
+				(hide yes)
+			)
+		)
+		(property "Value" "GND"
+			(at 312.42 54.356 0)
+			(effects
+				(font
+					(size 1.27 1.27)
+				)
+			)
+		)
+		(property "Footprint" ""
+			(at 312.42 49.53 0)
+			(effects
+				(font
+					(size 1.27 1.27)
+				)
+				(hide yes)
+			)
+		)
+		(property "Datasheet" ""
+			(at 312.42 49.53 0)
+			(effects
+				(font
+					(size 1.27 1.27)
+				)
+				(hide yes)
+			)
+		)
+		(property "Description" ""
+			(at 312.42 49.53 0)
+			(effects
+				(font
+					(size 1.27 1.27)
+				)
+				(hide yes)
+			)
+		)
+		(pin "1"
+		)
+		(instances
+			(project "DragonYUV"
+				(path "/60bcfc2a-b89b-48a4-90e1-5d504fe5d18a"
+					(reference "#PWR03")
+					(unit 1)
+				)
+			)
+		)
+	)
+	(symbol
 		(lib_id "74xx:74LS86")
 		(at 546.1 313.944 0)
@@
 			)
 		)
-		(property "Value" "AD624RJ"
+		(property "Value" "AD724RJ"
 			(at 406.0541 189.23 0)
 			(effects
@@
 	(symbol
 		(lib_id "power:GND")
+		(at 313.69 124.46 0)
+		(unit 1)
+		(exclude_from_sim no)
+		(in_bom yes)
+		(on_board yes)
+		(dnp no)
+		(fields_autoplaced yes)
+		(property "Reference" "#PWR046"
+			(at 313.69 130.81 0)
+			(effects
+				(font
+					(size 1.27 1.27)
+				)
+				(hide yes)
+			)
+		)
+		(property "Value" "GND"
+			(at 313.69 129.286 0)
+			(effects
+				(font
+					(size 1.27 1.27)
+				)
+			)
+		)
+		(property "Footprint" ""
+			(at 313.69 124.46 0)
+			(effects
+				(font
+					(size 1.27 1.27)
+				)
+				(hide yes)
+			)
+		)
+		(property "Datasheet" ""
+			(at 313.69 124.46 0)
+			(effects
+				(font
+					(size 1.27 1.27)
+				)
+				(hide yes)
+			)
+		)
+		(property "Description" ""
+			(at 313.69 124.46 0)
+			(effects
+				(font
+					(size 1.27 1.27)
+				)
+				(hide yes)
+			)
+		)
+		(pin "1"
+		)
+		(instances
+			(project "DragonYUV"
+				(path "/60bcfc2a-b89b-48a4-90e1-5d504fe5d18a"
+					(reference "#PWR046")
+					(unit 1)
+				)
+			)
+		)
+	)
+	(symbol
+		(lib_id "power:GND")
 		(at 322.58 97.79 0)
 		(unit 1)
@@
 					(unit 1)
 				)
+			)
+		)
+	)
+	(symbol
+		(lib_id "power:GND")
+		(at 313.69 91.44 0)
+		(unit 1)
+		(exclude_from_sim no)
+		(in_bom yes)
+		(on_board yes)
+		(dnp no)
+		(fields_autoplaced yes)
+		(property "Reference" "#PWR01"
+			(at 313.69 97.79 0)
+			(effects
+				(font
+					(size 1.27 1.27)
+				)
+				(hide yes)
+			)
+		)
+		(property "Value" "GND"
+			(at 313.69 96.266 0)
+			(effects
+				(font
+					(size 1.27 1.27)
+				)
+			)
+		)
+		(property "Footprint" ""
+			(at 313.69 91.44 0)
+			(effects
+				(font
+					(size 1.27 1.27)
+				)
+				(hide yes)
+			)
+		)
+		(property "Datasheet" ""
+			(at 313.69 91.44 0)
+			(effects
+				(font
+					(size 1.27 1.27)
+				)
+				(hide yes)
+			)
+		)
+		(property "Description" ""
+			(at 313.69 91.44 0)
+			(effects
+				(font
+					(size 1.27 1.27)
+				)
+				(hide yes)
+			)
+		)
+		(pin "1"
+		)
+		(instances
+			(project "DragonYUV"
+				(path "/60bcfc2a-b89b-48a4-90e1-5d504fe5d18a"
+					(reference "#PWR01")
+					(unit 1)
+				)

Commit message: reworked layout
Parts:
- removed TP4: TestPoint_Chroma, TestPoint:TestPoint_Pad_D1.0mm, symbol Connector:TestPoint_Probe
- U1: footprint Package_SO:SOIC-16_3.9x9.9mm_P1.27mm -> Package_SO:SOIC-16W_7.5x10.3mm_P1.27mm
Changed lines of the file:
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@@
 	(wire
 		(pts
-			(xy 140.208 46.99) (xy 144.018 46.99)
-		)
-		(stroke
-			(width 0)
-			(type default)
-		)
-	)
-	(wire
-		(pts
 			(xy 309.88 85.09) (xy 314.96 85.09)
 		)
@@
 		)
 	)
-	(global_label "CHB"
-		(shape output)
-		(at 140.208 46.99 180)
-		(fields_autoplaced yes)
-		(effects
-			(font
-				(size 1.27 1.27)
-			)
-			(justify right)
-		)
-		(property "Intersheetrefs" "${INTERSHEET_REFS}"
-			(at 134.0133 46.9106 0)
-			(effects
-				(font
-					(size 1.27 1.27)
-				)
-				(justify right)
-				(hide yes)
-			)
-		)
-	)
 	(global_label "CLK"
 		(shape input)
@@
 			)
 		)
-		(property "Footprint" "Package_SO:SOIC-16_3.9x9.9mm_P1.27mm"
+		(property "Footprint" "Package_SO:SOIC-16W_7.5x10.3mm_P1.27mm"
 			(at 402.59 204.47 0)
 			(effects
@@
 				)
 			)
-		)
-	)
-	(symbol
-		(lib_id "Connector:TestPoint_Probe")
-		(at 144.018 46.99 0)
-		(unit 1)
-		(exclude_from_sim no)
-		(in_bom yes)
-		(on_board yes)
-		(dnp no)
-		(fields_autoplaced yes)
-		(property "Reference" "TP4"
-			(at 147.828 44.1325 0)
-			(effects
-				(font
-					(size 1.27 1.27)
-				)
-				(justify left)
-			)
-		)
-		(property "Value" "TestPoint_Chroma"
-			(at 147.828 46.6725 0)
-			(effects
-				(font
-					(size 1.27 1.27)
-				)
-				(justify left)
-			)
-		)
-		(property "Footprint" "TestPoint:TestPoint_Pad_D1.0mm"
-			(at 149.098 46.99 0)
-			(effects
-				(font
-					(size 1.27 1.27)
-				)
-				(hide yes)
-			)
-		)
-		(property "Datasheet" "~"
-			(at 149.098 46.99 0)
-			(effects
-				(font
-					(size 1.27 1.27)
-				)
-				(hide yes)
-			)
-		)
-		(property "Description" ""
-			(at 144.018 46.99 0)
-			(effects
-				(font
-					(size 1.27 1.27)
-				)
-				(hide yes)
-			)
-		)
-		(pin "1"
-		)
-		(instances
-			(project "DragonYUV"
-				(path "/60bcfc2a-b89b-48a4-90e1-5d504fe5d18a"
-					(reference "TP4")
-					(unit 1)
-				)
-			)

Commit message: Clean up board Improve trace quality
Parts:
- added TP4: TestPoint_MuxX, TestPoint:TestPoint_Pad_D1.0mm, symbol Connector:TestPoint_Probe
Connections:
- net MUX X: now also TP4.1
Changed lines of the file:
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@@
 	(wire
 		(pts
+			(xy 139.7 48.26) (xy 143.51 48.26)
+		)
+		(stroke
+			(width 0)
+			(type default)
+		)
+	)
+	(wire
+		(pts
 			(xy 160.8074 377.6726) (xy 162.9664 377.6726)
 		)
@@
 	)
 	(global_label "MUX X"
+		(shape output)
+		(at 139.7 48.26 180)
+		(fields_autoplaced yes)
+		(effects
+			(font
+				(size 1.27 1.27)
+			)
+			(justify right)
+		)
+		(property "Intersheetrefs" "${INTERSHEET_REFS}"
+			(at 130.5463 48.26 0)
+			(effects
+				(font
+					(size 1.27 1.27)
+				)
+				(justify right)
+				(hide yes)
+			)
+		)
+	)
+	(global_label "MUX X"
 		(shape input)
 		(at 252.73 41.91 180)
@@
 					(unit 1)
 				)
+			)
+		)
+	)
+	(symbol
+		(lib_id "Connector:TestPoint_Probe")
+		(at 143.51 48.26 0)
+		(unit 1)
+		(exclude_from_sim no)
+		(in_bom yes)
+		(on_board yes)
+		(dnp no)
+		(fields_autoplaced yes)
+		(property "Reference" "TP4"
+			(at 147.32 45.4025 0)
+			(effects
+				(font
+					(size 1.27 1.27)
+				)
+				(justify left)
+			)
+		)
+		(property "Value" "TestPoint_MuxX"
+			(at 147.32 47.9425 0)
+			(effects
+				(font
+					(size 1.27 1.27)
+				)
+				(justify left)
+			)
+		)
+		(property "Footprint" "TestPoint:TestPoint_Pad_D1.0mm"
+			(at 148.59 48.26 0)
+			(effects
+				(font
+					(size 1.27 1.27)
+				)
+				(hide yes)
+			)
+		)
+		(property "Datasheet" "~"
+			(at 148.59 48.26 0)
+			(effects
+				(font
+					(size 1.27 1.27)
+				)
+				(hide yes)
+			)
+		)
+		(property "Description" ""
+			(at 143.51 48.26 0)
+			(effects
+				(font
+					(size 1.27 1.27)
+				)
+				(hide yes)
+			)
+		)
+		(pin "1"
+		)
+		(instances
+			(project "DragonYUV"
+				(path "/60bcfc2a-b89b-48a4-90e1-5d504fe5d18a"
+					(reference "TP4")
+					(unit 1)
+				)

Commit message: convert to cpld
Parts:
- removed C5: 100pF, Capacitor_SMD:C_0805_2012Metric_Pad1.18x1.45mm_HandSolder, symbol Device:C_Small
- removed C6: 180pF, Capacitor_SMD:C_0805_2012Metric_Pad1.18x1.45mm_HandSolder, symbol Device:C_Small
- removed C9: 0.01uF, Capacitor_SMD:C_0805_2012Metric_Pad1.18x1.45mm_HandSolder, symbol Device:C_Small
- removed IC10: 74HCT32, Package_SO:SOIC-14_3.9x8.7mm_P1.27mm, symbol 74xx:74LS32
- removed IC12: CD4053, Package_SO:SOIC-16_3.9x9.9mm_P1.27mm, symbol vdg:MC14053
- removed IC3: 74HCT00, Package_SO:SOIC-14_3.9x8.7mm_P1.27mm, symbol 74xx:74LS00
- removed IC4: 74HCT20, Package_SO:SOIC-14_3.9x8.7mm_P1.27mm, symbol 74xx:74LS20
- removed IC5: 74HCT86, Package_SO:SOIC-14_3.9x8.7mm_P1.27mm, symbol 74xx:74LS86
- removed IC6, IC8: 74HCT393, Package_SO:SOIC-14_3.9x8.7mm_P1.27mm, symbol 74xx:74LS393
- removed IC7: 74ALS74N, Package_SO:SOIC-14_3.9x8.7mm_P1.27mm, symbol 74xx:74LS74
- removed IC9: 74HCT390, Package_SO:SOIC-16_3.9x9.9mm_P1.27mm, symbol 74xx:74LS390
- removed R2: 12K, Resistor_SMD:R_0805_2012Metric_Pad1.20x1.40mm_HandSolder, symbol Device:R_Small
- removed R3: 8K2, Resistor_SMD:R_0805_2012Metric_Pad1.20x1.40mm_HandSolder, symbol Device:R_Small
- removed R4: 1K8, Resistor_SMD:R_0805_2012Metric_Pad1.20x1.40mm_HandSolder, symbol Device:R_Small
- removed TP7: TestPoint_LinePulse, TestPoint:TestPoint_Pad_D1.0mm, symbol Connector:TestPoint_Probe
- removed U2: 74AHC1G04, Package_TO_SOT_SMD:SOT-353_SC-70-5_Handsoldering, symbol 74xGxx:74AHC1G04
- added C16, C17, C18, C19: 0.1uF, Capacitor_SMD:C_0805_2012Metric_Pad1.18x1.45mm_HandSolder, symbol Device:C_Small
- added C20: 330pF, Capacitor_SMD:C_0805_2012Metric_Pad1.18x1.45mm_HandSolder, symbol Device:C_Small
- added IC11: 74LS123N, Package_SO:SOIC-16_3.9x9.9mm_P1.27mm, symbol 74xx:74LS123
- added J3: JTAG, Connector_PinHeader_1.27mm:PinHeader_2x05_P1.27mm_Vertical, symbol Connector_Generic:Conn_02x05_Odd_Even
- added R5: 27K, Resistor_SMD:R_0805_2012Metric_Pad1.20x1.40mm_HandSolder, symbol Device:R_Small
- added TP5: TestPoint_Green, TestPoint:TestPoint_Pad_D1.0mm, symbol Connector:TestPoint_Probe
- added TP6: TestPoint_Blue, TestPoint:TestPoint_Pad_D1.0mm, symbol Connector:TestPoint_Probe
- added U3: ATF1504ASL-xAx44, Package_QFP:TQFP-44_10x10mm_P0.8mm, symbol CPLD_Microchip:ATF1504ASL-xAx44
- C1: footprint Capacitor_SMD:CP_Elec_6.3x5.8 -> Capacitor_SMD:CP_Elec_4x5.4; DigiKey 732-8598-1-ND -> 732-6401-1-ND
- C10, C11, C12, C13, C15, C8: DigiKey (none) -> 732-6401-1-ND
- C14: value 52pF -> 51pF; DigiKey (none) -> 399-C0805C510F1GAC7800CT-ND
- C2: DigiKey 732-8598-1-ND -> 732-8254-1-ND
- C3, C7: DigiKey BC2662CT-ND -> 399-C0805C104M5RAC7800CT-ND
- C4: value 180pF -> 0.1uF; DigiKey BC1016CT-ND -> 399-C0805C104M5RAC7800CT-ND
- TP4: value TestPoint_MuxX -> TestPoint_Blue
- Y1: footprint Crystal:Crystal_SMD_0603-2Pin_6.0x3.5mm -> Crystal:Crystal_SMD_HC49-SD; DigiKey (none) -> XC1263CT-ND
Connections:
- net +5V: now also C4.2, C16.1, C17.1, C18.1, C19.1, IC11.10 (B), IC11.16 (VCC), IC11.3 (Clr), J3.4 (Pin_4), R5.2, U3.17 (VCC), U3.29 (VCC), U3.41 (VCC), U3.9 (VCC)
- net BLUE: now also TP4.1
- net CLK: now also U3.42 (I/O)
- net DA0: now also U3.43 (I/O)
- net GND: now also C4.1, C16.2, C17.2, C18.2, C19.2, C20.2, IC11.1 (A), IC11.11 (Clr), IC11.14 (Cext), IC11.6 (Cext), IC11.8 (GND), IC11.9 (A), J3.10 (Pin_10), J3.2 (Pin_2), U3.16 (GND), U3.24 (GND), U3.36 (GND), U3.4 (GND); no longer C4.2
- net GREEN: now also TP5.1
- net LUM: now also R8.2
- net LUM CONTROL: now also U3.33 (I/O)
- net RED: now also TP6.1
- net VCLK: now also U3.3 (I/O)
- net ~{FS}: now also U3.6 (I/O)
- net ~{HS}: now also U3.8 (I/O)
- net ~{NHS}: now also U3.44 (I/O)
- removed net MUX X: R8.2, TP4.1
- new net: C20.1, IC11.15 (RCext), R5.1
- new net Burst: IC11.2 (B), U3.31 (I/O)
- new net CHROME CONTROL: U3.30 (I/O)
- new net DA0': U3.2 (I/O)
- new net E: U3.10 (I/O)
- new net PadLuma: U3.34 (I/O)
- new net PhaseT: IC11.4 (~{Q}), U3.11 (I/O)
- new net TCK: J3.1 (Pin_1), U3.26 (I/O/TCK)
- new net TDI: J3.9 (Pin_9), U3.1 (I/O/TDI)
- new net TDO: J3.3 (Pin_3), U3.32 (I/O/TDO)
- new net TMS: J3.5 (Pin_5), U3.7 (I/O/TMS)
- new net ~{RESET}: J3.6 (Pin_6)
- no-connect marks 52 -> 44
Other:
- note added: "3us PULSE (APPROX)"
- note removed: "24 LINE DELAY"
- note removed: "DIVIDE BY 50"
- note removed: "DIVIDE VCLK BY 228 TO CREATE LINE PULSE FREQUENCY"
- note removed: "MUX X = SELECT LUMA SIGNAL FROM VDG OR EXTRA SYNCS FROM LINE PULSE CIRCUIT MUX Y = SUBSTITUTE ØB FOR ØA DURING BACK PORCH SO THAT CHROMA BURST IS INCLUDED IN PHASE ALTERNATION MUX Z = ALTERNATING PHASE"
- note removed: "OUTPUT LOW ON COUNT 0-15 LINE PULSE WIDTH = 4.5us"
- note removed: "STEER VCLK TO VDG OR LINE PULSE CIRCUIT"

Commit message: update design to provide ntsc and pal switching
Parts:
- added C5, C6: 220uF, Capacitor_SMD:CP_Elec_4x5.4, symbol Device:C_Polarized_Small
- added J4: SVid, Connector_PinHeader_2.54mm:PinHeader_1x04_P2.54mm_Vertical, symbol Connector:Conn_01x04_Pin
- added JP1: Video Clock, Jumper:SolderJumper-3_P1.3mm_Open_Pad1.0x1.5mm_NumberLabels, symbol Jumper:SolderJumper_3_Open
- added JP2: Video HS, Jumper:SolderJumper-3_P1.3mm_Open_Pad1.0x1.5mm_NumberLabels, symbol Jumper:SolderJumper_3_Open
- added JP3: Video Format, Jumper:SolderJumper-3_P1.3mm_Open_Pad1.0x1.5mm_NumberLabels, symbol Jumper:SolderJumper_3_Open
- added R2, R3: 75R, Resistor_SMD:R_0805_2012Metric_Pad1.20x1.40mm_HandSolder, symbol Device:R_Small
- added R4, R6: 10K, Resistor_SMD:R_0805_2012Metric_Pad1.20x1.40mm_HandSolder, symbol Device:R_Small
- C15: value 10uF -> 220uF
- U1: value AD724RJ -> AD724JR
- Y1: footprint Crystal:Crystal_SMD_HC49-SD -> Crystal:Crystal_HC18-U_Vertical
Connections:
- net +5V: now also R4.2, R6.1; no longer U1.5 (CE)
- net CLK: now also JP1.2 (C); no longer U3.42 (I/O)
- net GND: now also J4.1 (Pin_1), J4.4 (Pin_4), JP3.1 (A); no longer U1.1 (NTSC/PAL)
- net VCLK: now also JP1.3 (B)
- net ~{HS}: now also JP2.3 (B)
- net ~{NHS}: now also JP2.2 (C); no longer U3.44 (I/O)
- net at U1.11 (LUM_OUT): now also C6.1
- net at U1.9 (CHROM_OUT): now also C5.1
- new net: C6.2, R3.2
- new net: JP3.2 (C), U1.1 (NTSC/PAL)
- new net: JP3.3 (B), R4.1
- new net: C5.2, R2.2
- new net: R6.2, U1.5 (CE)
- new net CHROMA OUT: J4.3 (Pin_3), R2.1
- new net CLK': JP1.1 (A), U3.42 (I/O)
- new net LUMA OUT: J4.2 (Pin_2), R3.1
- new net ~{HS'}: JP2.1 (A), U3.44 (I/O)
- no-connect marks 44 -> 42
Other:
- moved on the sheet: C15, C16, C17, C18, C19, C20, IC11A, IC11B, J3, R1, R5, U3
